File: projpcb.kicad_pcb (KiCad board)
At the start: 2 copper layers, 34 parts, among them CON1 BARREL_JACK, CON2 BARREL_JACK, P1 CONN_01X02, P2 CONN_01X02, Q1 SFH3711, Q10 SFH3711, Q11 SFH3711, Q12 SFH3711, Q13 SFH3711, Q14 SFH3711, Q15 SFH3711, Q16 Q_NMOS_GSD, Q2 SFH3711, Q3 SFH3711, Q4 SFH3711, Q5 SFH3711, Q6 SFH3711, Q7 SFH3711, Q8 SFH3711, Q9 SFH3711, U1 Teensy_3.1, U2 LM358, U3 CD74HC4067, U4 CL520

Commit message: BoardV2
Parts:
- moved C1 16.9 mm to (146.4, 114.0), turned to 180 degrees
- moved C2 16.9 mm to (146.4, 109.2), turned to 180 degrees
- moved R2 5.06 mm to (154.8, 129.9), turned to 0 degrees
- turned C3 to 0 degrees
- turned Q11 to 180 degrees
Routing:
- net /Phototransistors/S13: track 0.00 -> 82.4 mm
- net /Phototransistors/S14: track 0.00 -> 82.2 mm
- net /Phototransistors/S12: track 0.00 -> 81.9 mm
- net /Phototransistors/S15: track 0.00 -> 81.8 mm
- net /Phototransistors/S11: track 0.00 -> 81.7 mm
- net T3: track 0.00 -> 51.0 mm
- net T2: track 0.00 -> 49.1 mm
- net HEAT: track 0.00 -> 44.0 mm
- net VIN: track 0.00 -> 33.3 mm
- net Net-(R1-Pad1): track 0.00 -> 29.4 mm
- net Net-(CON2-Pad2): track 0.00 -> 25.8 mm
- net T5: track 0.00 -> 24.2 mm
- net Net-(RV2-Pad1): track 15.0 -> 35.1 mm
- net T6: track 0.00 -> 18.0 mm
- net Net-(P2-Pad2): track 0.00 -> 17.3 mm
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Other:
- board outline added: 130 x 70 mm
