File: DONNE.kicad_pcb (KiCad board)
At the start: 2 copper layers, 110 x 72.5 mm, 40 parts, among them CON1 BARREL_JACK, CON2 BARREL_JACK, P1 CONN_01X02, P2 CONN_01X02, Q1 SFH3711, Q10 SFH3711, Q11 SFH3711, Q12 SFH3711, Q13 SFH3711, Q14 SFH3711, Q15 SFH3711, Q16 Q_NMOS_GSD, Q2 SFH3711, Q3 SFH3711, Q4 SFH3711, Q5 SFH3711, Q6 SFH3711, Q7 SFH3711, Q8 SFH3711, Q9 SFH3711, U1 Teensy_3.1, U2 LM358, U3 CD74HC4067, U4 CL520

Commit message: PCB
Parts:
- C1: moved to B.Cu
Connections:
- C1 pad 2: Net-(C1-Pad2) -> GNDA
- U3 pad 12: Net-(C1-Pad2) -> GNDA
Routing:
- net GNDA: track 61.4 -> 119.5 mm, vias 0 -> 2
- net /Phototransistors/S2: track 41.3 -> 20.6 mm
- net Net-(C1-Pad2): track 14.6 -> 0.00 mm
- net +3V3: track 224.5 -> 223.4 mm
Other:
- board text added: "1k"

Commit message: PCB
Parts:
- R1: moved to B.Cu
- moved C2 9.40 mm to (168.0, 74.0), turned to 0 degrees
- moved R1 2.49 mm to (177.0, 65.0), turned to 90 degrees
Routing:
- net GNDA: track 119.5 -> 6.05 mm, vias 2 -> 0
- net +3V3: track 223.4 -> 218.6 mm
- net Net-(D2-Pad1): track 2.68 -> 5.98 mm
- net Net-(R1-Pad1): track 22.8 -> 21.1 mm
Changed lines of the file:
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@@
   (general
     (links 83)
-    (no_connects 2)
+    (no_connects 4)
     (area 137.449999 52.449999 247.550001 125.050001)
     (thickness 1.6)
     (drawings 5)
-    (tracks 244)
+    (tracks 217)
     (zones 0)
     (modules 40)
@@
   (page A4)
   (layers
-    (0 F.Cu signal hide)
+    (0 F.Cu signal)
     (31 B.Cu signal)
     (32 B.Adhes user)
@@
   )
   (module Capacitors_SMD:C_0805_HandSoldering (layer B.Cu)
-    (at 158.6 73.8 270)
+    (at 168 74)
     (descr "Capacitor SMD 0805, hand soldering")
     (tags "capacitor 0805")
     (attr smd)
-    (fp_text reference C2 (at 0 2.1 270) (layer B.SilkS)
-      (effects (font (size 1 1) (thickness 0.15)) (justify mirror))
-    )
-    (fp_text value 100nF (at 0 -2.1 270) (layer B.Fab)
+    (fp_text reference C2 (at 0 2.1) (layer B.SilkS)
+      (effects (font (size 1 1) (thickness 0.15)) (justify mirror))
+    )
+    (fp_text value 100nF (at 0 -2.1) (layer B.Fab)
       (effects (font (size 1 1) (thickness 0.15)) (justify mirror))
     )
@@
     (fp_line (start 0.5 0.85) (end -0.5 0.85) (layer B.SilkS) (width 0.15))
     (fp_line (start -0.5 -0.85) (end 0.5 -0.85) (layer B.SilkS) (width 0.15))
-    (pad 1 smd rect (at -1.25 0 270) (size 1.5 1.25) (layers B.Cu B.Paste B.Mask)
-      (net 1 +3V3))
-    (pad 2 smd rect (at 1.25 0 270) (size 1.5 1.25) (layers B.Cu B.Paste B.Mask)
+    (pad 1 smd rect (at -1.25 0) (size 1.5 1.25) (layers B.Cu B.Paste B.Mask)
+      (net 1 +3V3))
+    (pad 2 smd rect (at 1.25 0) (size 1.5 1.25) (layers B.Cu B.Paste B.Mask)
       (net 2 GNDA))
     (model Capacitors_SMD.3dshapes/C_0805_HandSoldering.wrl
@@
     )
   )
-  (module Resistors_SMD:R_0805_HandSoldering (layer F.Cu)
-    (at 174.6 64.35 270)
-    (descr "Resistor SMD 0805, hand soldering")
-    (tags "resistor 0805")
-    (attr smd)
-    (fp_text reference R1 (at 0 -2.1 270) (layer F.SilkS)
-      (effects (font (size 1 1) (thickness 0.15)))
-    )
-    (fp_text value 1K (at 0 2.1 270) (layer F.Fab)
-      (effects (font (size 1 1) (thickness 0.15)))
-    )
-    (fp_line (start -2.4 -1) (end 2.4 -1) (layer F.CrtYd) (width 0.05))
-    (fp_line (start -2.4 1) (end 2.4 1) (layer F.CrtYd) (width 0.05))
-    (fp_line (start -2.4 -1) (end -2.4 1) (layer F.CrtYd) (width 0.05))
-    (fp_line (start 2.4 -1) (end 2.4 1) (layer F.CrtYd) (width 0.05))
-    (fp_line (start 0.6 0.875) (end -0.6 0.875) (layer F.SilkS) (width 0.15))
-    (fp_line (start -0.6 -0.875) (end 0.6 -0.875) (layer F.SilkS) (width 0.15))
-    (pad 1 smd rect (at -1.35 0 270) (size 1.5 1.3) (layers F.Cu F.Paste F.Mask)
+  (module Resistors_SMD:R_0805_HandSoldering (layer B.Cu)
+    (at 177 65 90)
+    (descr "Resistor SMD 0805, hand soldering")
+    (tags "resistor 0805")
+    (attr smd)
+    (fp_text reference R1 (at 0 2.1 90) (layer B.SilkS)
+      (effects (font (size 1 1) (thickness 0.15)) (justify mirror))
+    )
+    (fp_text value 1K (at 0 -2.1 90) (layer B.Fab)
+      (effects (font (size 1 1) (thickness 0.15)) (justify mirror))
+    )
+    (fp_line (start -2.4 1) (end 2.4 1) (layer B.CrtYd) (width 0.05))
+    (fp_line (start -2.4 -1) (end 2.4 -1) (layer B.CrtYd) (width 0.05))
+    (fp_line (start -2.4 1) (end -2.4 -1) (layer B.CrtYd) (width 0.05))
+    (fp_line (start 2.4 1) (end 2.4 -1) (layer B.CrtYd) (width 0.05))
+    (fp_line (start 0.6 -0.875) (end -0.6 -0.875) (layer B.SilkS) (width 0.15))
+    (fp_line (start -0.6 0.875) (end 0.6 0.875) (layer B.SilkS) (width 0.15))
+    (pad 1 smd rect (at -1.35 0 90) (size 1.5 1.3) (layers B.Cu B.Paste B.Mask)
       (net 32 "Net-(R1-Pad1)"))
-    (pad 2 smd rect (at 1.35 0 270) (size 1.5 1.3) (layers F.Cu F.Paste F.Mask)
+    (pad 2 smd rect (at 1.35 0 90) (size 1.5 1.3) (layers B.Cu B.Paste B.Mask)
       (net 2 GNDA))
     (model Resistors_SMD.3dshapes/R_0805_HandSoldering.wrl
@@
   (segment (start 159.5 77.75) (end 162.38 74.87) (width 0.25) (layer F.Cu) (net 1))
   (segment (start 160.54 112.46) (end 157.26 112.46) (width 0.25) (layer F.Cu) (net 1))
-  (segment (start 162.38 70) (end 161.15 70) (width 0.25) (layer B.Cu) (net 1))
-  (segment (start 161.15 70) (end 158.6 72.55) (width 0.25) (layer B.Cu) (net 1))
   (segment (start 163.75 110) (end 163 110) (width 0.25) (layer F.Cu) (net 1))
   (segment (start 163 110) (end 160.54 112.46) (width 0.25) (layer F.Cu) (net 1))
@@
   (segment (start 163.75 110) (end 163.75 115) (width 0.25) (layer F.Cu) (net 1))
   (segment (start 163.75 100) (end 163.75 105) (width 0.25) (layer F.Cu) (net 1))
-  (segment (start 170 77.62) (end 173.13 77.62) (width 0.25) (layer F.Cu) (net 2))
-  (segment (start 195.75 87.5) (end 196 87.25) (width 0.25) (layer B.Cu) (net 2))
-  (segment (start 196 87.25) (end 196 75.5) (width 0.25) (layer B.Cu) (net 2))
-  (segment (start 196 75.5) (end 190.5 70) (width 0.25) (layer B.Cu) (net 2))
-  (segment (start 190.5 70) (end 181 70) (width 0.25) (layer B.Cu) (net 2))
-  (segment (start 181 70) (end 174.25 76.75) (width 0.25) (layer B.Cu) (net 2))
-  (segment (start 195.75 87.5) (end 195 87.5) (width 0.25) (layer B.Cu) (net 2))
-  (segment (start 174 76.75) (end 174.25 76.75) (width 0.25) (layer B.Cu) (net 2))
-  (segment (start 173.5 77.25) (end 174 76.75) (width 0.25) (layer B.Cu) (net 2))
-  (via (at 173.5 77.25) (size 0.6) (drill 0.4) (layers F.Cu B.Cu) (net 2))
-  (segment (start 173.13 77.62) (end 173.5 77.25) (width 0.25) (layer F.Cu) (net 2))
-  (segment (start 195 94) (end 195 95.69) (width 0.25) (layer F.Cu) (net 2))
-  (segment (start 195 95.69) (end 199 99.69) (width 0.25) (layer F.Cu) (net 2))
-  (segment (start 195 87.5) (end 195 94) (width 0.25) (layer B.Cu) (net 2))
-  (via (at 195 94) (size 0.6) (drill 0.4) (layers F.Cu B.Cu) (net 2))
   (segment (start 161.65 119) (end 161.26 119) (width 0.25) (layer B.Cu) (net 2))
   (segment (start 161.26 119) (end 157.26 115) (width 0.25) (layer B.Cu) (net 2))
-  (segment (start 174.6 65.7) (end 174.6 73.02) (width 0.25) (layer F.Cu) (net 2))
-  (segment (start 174.6 73.02) (end 170 77.62) (width 0.25) (layer F.Cu) (net 2))
-  (segment (start 158.6 75.05) (end 158.6 74.6) (width 0.25) (layer B.Cu) (net 2))
-  (segment (start 158.6 74.6) (end 149 65) (width 0.25) (layer B.Cu) (net 2))
-  (segment (start 154.13 58) (end 156.98 60.85) (width 0.25) (layer B.Cu) (net 2))
-  (segment (start 151 58) (end 154.13 58) (width 0.25) (layer B.Cu) (net 2))
-  (segment (start 149 60) (end 151 58) (width 0.25) (layer B.Cu) (net 2))
-  (segment (start 149 65) (end 149 60) (width 0.25) (layer B.Cu) (net 2))
-  (segment (start 158.6 75.05) (end 167.43 75.05) (width 0.25) (layer B.Cu) (net 2))
-  (segment (start 167.43 75.05) (end 170 77.62) (width 0.25) (layer B.Cu) (net 2))
   (segment (start 148.20014 73) (end 148.20014 88) (width 1) (layer F.Cu) (net 4))
   (segment (start 152.4 82.90114) (end 152.4 92.1) (width 1) (layer F.Cu) (net 6))
@@
   (segment (start 170 96.75) (end 170 118.5) (width 0.25) (layer F.Cu) (net 10))
   (segment (start 162.85 89.6) (end 170 96.75) (width 0.25) (layer F.Cu) (net 10))
+  (segment (start 186.35 115) (end 186.35 118.14902) (width 0.25) (layer F.Cu) (net 11))
+  (segment (start 186.35 118.14902) (end 186.45098 118.25) (width 0.25) (layer F.Cu) (net 11))
   (segment (start 186.35 115) (end 186.35 117.39902) (width 0.25) (layer F.Cu) (net 11))
   (segment (start 186.35 117.39902) (end 186.45098 117.5) (width 0.25) (layer F.Cu) (net 11))
@@
   (segment (start 153.35 79.89886) (end 157.29886 79.89886) (width 0.25) (layer F.Cu) (net 31))
   (segment (start 167.8 92.52) (end 172.5 97.22) (width 0.25) (layer F.Cu) (net 31))
+  (segment (start 177 66.35) (end 169.6 66.35) (width 0.25) (layer B.Cu) (net 32))
+  (segment (start 169.6 66.35) (end 166.99 63.74) (width 0.25) (layer B.Cu) (net 32))
   (segment (start 164.45 61.2) (end 166.99 63.74) (width 0.25) (layer F.Cu) (net 32))
-  (segment (start 174.6 63) (end 174 63) (width 0.25) (layer F.Cu) (net 32))
-  (segment (start 174 63) (end 170 59) (width 0.25) (layer F.Cu) (net 32))
-  (segment (start 170 59) (end 166.65 59) (width 0.25) (layer F.Cu) (net 32))
-  (segment (start 166.65 59) (end 164.45 61.2) (width 0.25) (layer F.Cu) (net 32))
   (segment (start 166.99 63.74) (end 166.99 69.53) (width 0.25) (layer F.Cu) (net 32))
   (segment (start 166.99 69.53) (end 167.46 70) (width 0.25) (layer F.Cu) (net 32))
@@
     (polygon
       (pts
-        (xy 201 121) (xy 150 121) (xy 150 57) (xy 201 57) (xy 201 121)
+        (xy 211 125) (xy 138 125) (xy 138 53) (xy 211 53) (xy 211 125)
       )
     )

Commit message: VERSION ONE - Sent for manufacturegit add -Agit add -A
Parts:
- removed RV2: POT, Potentiometers:Potentiometer_Trimmer-Suntan-TSR-3386P
Connections:
- C1 pad 2: GNDA -> GND
- C2 pad 2: GNDA -> GND
- R1 pad 2: GNDA -> GND
- R2 pad 2: GNDA -> GND
- U1 pad 25: GNDA -> GND
- U2 pad 8: GNDA -> GND
- U3 pad 12: GNDA -> GND
Routing:
- net GND: track 0.00 -> 207.5 mm, vias 0 -> 36
- net +3V3: track 218.6 -> 238.8 mm, vias 2 -> 5
- net GNDA: track 6.05 -> 0.00 mm
- added copper zone on B.Cu, net GND
- removed copper zone on B.Cu, net GNDA
